File: kicad/solar_bird_pcb_01.kicad_pcb (KiCad board)
At the start: 2 copper layers, 40 x 24 mm, 8 parts, among them J1 Conn_01x01, J2 Conn_01x01, J3 Conn_01x01, J4 Conn_01x01, J5 Conn_02x03_Odd_Even, U1 ATtiny13V-10PU

Commit message: Bird pcb layout
Routing:
- net GND: track 21.6 -> 0.00 mm
- net /MISO: track 20.7 -> 10.8 mm
- net /SCK: track 14.0 -> 6.08 mm
- net /MOSI: track 24.0 -> 20.2 mm
Other:
- board text added: "1"
